Commit message: urdf updates

File: src/transformer_description/urdf/transformer.urdf.xacro (robot description, xacro)
@@ -8,5 +8,6 @@
         <mesh filename="package://transformer_description/model/transformer_model.stl" scale="1 1 1"/>
       </geometry>
-      <origin xyz="0 0 0" rpy="0 0 0"/>
+      <!-- Rotate model 90 degrees around Z axis -->
+      <origin xyz="0 0 0" rpy="0 0 1.57079632679"/>
       <material name="gray"><color rgba="0.6 0.6 0.6 1.0"/></material>
     </visual>
@@ -16,5 +17,6 @@
         <mesh filename="package://transformer_description/model/transformer_model.stl" scale="1 1 1"/>
       </geometry>
-      <origin xyz="0 0 0" rpy="0 0 0"/>
+      <!-- Match visual rotation for collision -->
+      <origin xyz="0 0 0" rpy="0 0 1.57079632679"/>
     </collision>
     <inertial>
@@ -24,11 +26,11 @@
   </link>
   <!-- Parameters for sensor poses (placeholders; override via launch or set params) -->
-  <xacro:property name="msp_imu_xyz" value="0.0 0.0 0.1"/>
+  <xacro:property name="msp_imu_xyz" value="0.0 0.0 0.14"/>
   <xacro:property name="msp_imu_rpy" value="0.0 0.0 0.0"/>
-  <xacro:property name="n100_imu_xyz" value="0.0 0.0 0.12"/>
+  <xacro:property name="n100_imu_xyz" value="0.0 0.0 0.16"/>
   <xacro:property name="n100_imu_rpy" value="0.0 0.0 0.0"/>
-  <xacro:property name="gps_xyz" value="0.2 0.0 0.2"/>
+  <xacro:property name="gps_xyz" value="0.1415 0.0 0.2"/>
   <xacro:property name="gps_rpy" value="0.0 0.0 0.0"/>
-  <xacro:property name="d435i_xyz" value="0.25 0.0 0.2"/>
+  <xacro:property name="d435i_xyz" value="0.175 0.0 0.2"/>
   <xacro:property name="d435i_rpy" value="0.0 0.0 0.0"/>
   <!-- MSP IMU link -->

Commit message: updated stats

File: src/transformer_description/urdf/transformer.urdf.xacro (robot description, xacro)
@@ -20,8 +20,4 @@
       <origin xyz="0 0 0" rpy="0 0 1.57079632679"/>
     </collision>
-    <inertial>
-      <mass value="5.0"/>
-      <inertia ixx="0.1" ixy="0.0" ixz="0.0" iyy="0.1" iyz="0.0" izz="0.1"/>
-    </inertial>
   </link>
   <!-- Parameters for sensor poses (placeholders; override via launch or set params) -->

Commit message: added comments for documentation

File: src/transformer_description/urdf/transformer.urdf.xacro (robot description, xacro)
@@ -72,6 +72,6 @@
     <origin xyz="${gps_xyz}" rpy="${gps_rpy}"/>
   </joint>
-  <!-- Intel RealSense D435i base link (matches realsense2_camera frame name) -->
-  <link name="D435I_link">
+  <!-- Intel RealSense D435i base link (aligned with realsense2_camera frame names) -->
+  <link name="camera_D435I_link">
     <visual>
       <geometry>
@@ -81,7 +81,7 @@
     </visual>
   </link>
-  <joint name="D435I_joint" type="fixed">
+  <joint name="camera_D435I_joint" type="fixed">
     <parent link="base_link"/>
-    <child link="D435I_link"/>
+    <child link="camera_D435I_link"/>
     <origin xyz="${d435i_xyz}" rpy="${d435i_rpy}"/>
   </joint>
